Commit message: update urdf

File: arm_description/urdf/arm.urdf (robot description, URDF)
Before this commit: robot arm, 6 links, 5 joints
Links:
- link frontal_arm: geometry collision mesh filename=package://arm_description/meshes/frontal_arm.stl; visual mesh filename=package://arm_description/meshes/frontal_arm.stl
Joints:
- joint elbow_joint: origin xyz=0 0 0.2 rpy=0 1.5707 0 -> xyz=-0.2 0 0.015 rpy=0 0 1.5707
- joint wrist_joint: origin xyz=0 0 0.15 rpy=1.5707 0 1.5707 -> xyz=0 0.15 -0.015 rpy=0 0 -1.5707; parent elbow -> frontal_arm
